Commit message: Final?

File: sim_ws/src/agc_golfcart_sim/models/golfcart/model.xacro.urdf (robot description, URDF)
Before this commit: robot uwf_golfcart, 12 links, 11 joints
Links:
- link steering_input_link: mass 0.01 -> 20.0
Joints:
- joint steering_input_joint: limit lower=-0.785 upper=0.785 effort=100 velocity=1.0 -> lower=-0.785 upper=0.785 effort=100 velocity=0.5
